File: PCB/hydropad.kicad_sch (KiCad schematic)
At the start: 14 parts, among them SW1 SW_Push, SW2 SW_Push, SW3 SW_Push, SW4 SW_Push, SW5 SW_Push, SW7 RotaryEncoder_Switch, U1 MODULE-SEEEDUINO-XIAO

Commit message: Add some CAD data
Other:
- moved on the sheet: D1, D2, D3, D4, D5, D6, DISPLAY, SW1, SW2, SW3, SW4, SW5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
